File: kicad/STR500_v1.2/STR500_v1.2.kicad_sch (KiCad schematic)
At the start: 21 parts, among them J1 FootswitchMolex, J2 Barrel_Jack, J3 AudioOutL, J4 AudioOutR, J5 AudioInR, J6 AudioInL, SW1 PitchOn, SW2 PowerSwitch, SW3 FilterOn

Commit message: rerouted as 2L
Parts:
- GameTrak1: value ~ -> (none)
Other:
- note added: "220u is too much decoupling for USB, i know this is a barrel jack but qualify your power supply with a cheap scope if you want to understand it better"
- note added: "potentially add a pi filter / series ferrite bead here."
- note added: "you have plenty of space on the board, you could add 2.54mm perfboard for experimenting with SMT components"
