File: kicad/STR500_v1.2/STR500_v1.2.kicad_pcb (KiCad board)
At the start: 4 copper layers, 65 x 100 mm, 23 parts, among them J1 FootswitchMolex, J2 Barrel_Jack, J3 AudioOutL, J4 AudioOutR, J5 AudioInR, J6 AudioInL, SW1 PitchOn, SW2 PowerSwitch, SW3 FilterOn

Commit message: rerouted as 2L
Parts:
- moved C1 8.38 mm to (114.5, 68.0)
- moved C2 3.61 mm to (119.0, 68.0), turned to -90 degrees
Routing:
- net +5V: track 36.4 -> 43.6 mm
- net /BT1: track 42.4 -> 35.5 mm
- net Net-(D1-A): track 25.8 -> 21.2 mm
- net +3.3V: track 33.8 -> 38.0 mm
- net /Pot1: track 33.8 -> 31.1 mm
- net /outL: track 24.6 -> 26.2 mm
- net /Sw2: track 65.6 -> 67.2 mm
- net /BT4: track 15.7 -> 17.1 mm
- net /inL: track 26.3 -> 25.8 mm
- net /Sw1: vias 0 -> 1
- net GND: vias 0 -> 40
- added copper zone on B.Cu, net GND
- added copper zone on F.Cu, net GND
- removed copper zone on In2.Cu, net GND
Other:
- copper layers 4 -> 2

Commit message: small changes to PCB, renaming JSON file
Other:
- board text added: "August 2026 / Yann Seznec Impractical Devices"
- board text added: "GND"
- board text added: "bridge for use without footswitch sockets"
- board text removed: "May 2026 / Yann Seznec Impractical Devices"
- board text removed: "bridge to use without footswitch sockets"

Commit message: cosmetic update to PCB
Other:
- board text added: "October 2026 / Yann Seznec"
- board text removed: "August 2026 / Yann Seznec Impractical Devices"
